File: Hardware/KiCad/Schematic-PCB/Master Chess Board/Clock PCB.kicad_sch (KiCad schematic)
At the start: 10 parts, among them J7 ZF1-15-02-X-WT-X

Commit message: Small iteration
Parts:
- DS2: value OLED_128X64_1.3_I2C -> OLED_128X32_2.23_I2C; footprint OLED_128X64_1.3_I2C:LCD_OLED_128X64_1.3_I2C -> OLED_128X64_1.3_I2C:LCD_OLED_128X32_2.23_I2C
Other:
- note added: "Needs to be 2.23" OLED screen"
- note removed: "Needs to be 2.42" OLED screen"
Changed lines of the file:
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@@
 	(text "SDA: GPIO 8   SCL: GPIO 9"
 		(exclude_from_sim no)
-		(at 109.728 91.186 0)
+		(at 109.728 93.218 0)
 		(effects
 			(font
@@
 		)
 	)
-	(text "Needs to be 2.42\" OLED screen\n"
+	(text "Needs to be 2.23\" OLED screen\n"
 		(exclude_from_sim no)
 		(at 184.15 134.62 0)
@@
 	)
 	(junction
-		(at 101.6 121.92)
+		(at 138.43 100.33)
 		(diameter 0)
 		(color 0 0 0 0)
 	)
 	(junction
-		(at 179.07 114.3)
+		(at 101.6 121.92)
 		(diameter 0)
 		(color 0 0 0 0)
 	)
 	(junction
-		(at 143.51 100.33)
+		(at 179.07 114.3)
 		(diameter 0)
 		(color 0 0 0 0)
@@
 	(wire
 		(pts
+			(xy 138.43 91.44) (xy 142.24 91.44)
+		)
+		(stroke
+			(width 0)
+			(type default)
+		)
+	)
+	(wire
+		(pts
 			(xy 194.31 97.79) (xy 97.79 97.79)
 		)
@@
 	(wire
 		(pts
-			(xy 137.16 119.38) (xy 143.51 119.38)
+			(xy 138.43 100.33) (xy 138.43 91.44)
 		)
 		(stroke
@@
 	(wire
 		(pts
-			(xy 143.51 95.25) (xy 143.51 100.33)
+			(xy 137.16 119.38) (xy 143.51 119.38)
 		)
 		(stroke
@@
 	(wire
 		(pts
-			(xy 148.59 100.33) (xy 143.51 100.33)
+			(xy 96.52 129.54) (xy 101.6 129.54)
 		)
 		(stroke
@@
 	(wire
 		(pts
-			(xy 96.52 129.54) (xy 101.6 129.54)
+			(xy 104.14 114.3) (xy 104.14 121.92)
 		)
 		(stroke
@@
 	(wire
 		(pts
-			(xy 104.14 114.3) (xy 104.14 121.92)
+			(xy 179.07 128.27) (xy 148.59 128.27)
 		)
 		(stroke
@@
 	(wire
 		(pts
-			(xy 179.07 128.27) (xy 148.59 128.27)
+			(xy 134.62 100.33) (xy 138.43 100.33)
 		)
 		(stroke
@@
 	(wire
 		(pts
-			(xy 134.62 100.33) (xy 143.51 100.33)
+			(xy 101.6 121.92) (xy 92.71 121.92)
 		)
 		(stroke
@@
 	(wire
 		(pts
-			(xy 101.6 121.92) (xy 92.71 121.92)
+			(xy 138.43 100.33) (xy 148.59 100.33)
 		)
 		(stroke
@@
 	(hierarchical_label "GND"
 		(shape output)
-		(at 143.51 96.52 0)
+		(at 142.24 91.44 0)
 		(effects
 			(font
@@
 		)
 		(instances
+			(project "Clock PCB"
+				(path "/7f3c47f2-1a05-49da-84f6-af3328144f29"
+					(reference "100nF70")
+					(unit 1)
+				)
+			)
 			(project "StockfishChess"
 				(path "/e9cb1197-186c-4036-91fc-6928f1600b5f/83544a14-6c08-41fb-841d-407afd354856"
@@
 	(symbol
 		(lib_id "power:GND")
-		(at 95.25 88.9 90)
+		(at 95.25 88.9 0)
 		(unit 1)
 		(body_style 1)
@@
 		(fields_autoplaced yes)
 		(property "Reference" "#PWR064"
-			(at 101.6 88.9 0)
+			(at 95.25 95.25 0)
 			(hide yes)
 			(show_name no)
@@
 		)
 		(property "Value" "GND"
-			(at 99.06 88.8999 90)
+			(at 97.79 90.1699 0)
 			(show_name no)
 			(do_not_autoplace no)
@@
 					(size 1.27 1.27)
 				)
-				(justify right)
+				(justify left)
 			)
 		)
@@
 		)
 		(instances
+			(project "Clock PCB"
+				(path "/7f3c47f2-1a05-49da-84f6-af3328144f29"
+					(reference "#PWR064")
+					(unit 1)
+				)
+			)
 			(project "StockfishChess"
 				(path "/e9cb1197-186c-4036-91fc-6928f1600b5f/83544a14-6c08-41fb-841d-407afd354856"
@@
 		)
 		(instances
+			(project "Clock PCB"
+				(path "/7f3c47f2-1a05-49da-84f6-af3328144f29"
+					(reference "#PWR075")
+					(unit 1)
+				)
+			)
 			(project "StockfishChess"
 				(path "/e9cb1197-186c-4036-91fc-6928f1600b5f/83544a14-6c08-41fb-841d-407afd354856"
@@
 	(symbol
 		(lib_id "power:+3.3V")
-		(at 95.25 86.36 270)
+		(at 95.25 86.36 0)
 		(unit 1)
 		(body_style 1)
@@
 		(fields_autoplaced yes)
 		(property "Reference" "#PWR063"
-			(at 91.44 86.36 0)
+			(at 95.25 90.17 0)
 			(hide yes)
 			(show_name no)
@@
 		)
 		(property "Value" "+3.3V"
-			(at 99.06 86.3599 90)
+			(at 97.79 85.0899 0)
 			(show_name no)
 			(do_not_autoplace no)
@@
 		)
 		(instances
+			(project "Clock PCB"
+				(path "/7f3c47f2-1a05-49da-84f6-af3328144f29"
+					(reference "#PWR063")
+					(unit 1)
+				)
+			)
 			(project "StockfishChess"
 				(path "/e9cb1197-186c-4036-91fc-6928f1600b5f/83544a14-6c08-41fb-841d-407afd354856"
@@
 	(symbol
 		(lib_id "power:GND")
-		(at 143.51 95.25 180)
+		(at 142.24 91.44 0)
 		(unit 1)
 		(body_style 1)
@@
 		(in_pos_files yes)
 		(dnp no)
-		(fields_autoplaced yes)
 		(property "Reference" "#PWR065"
-			(at 143.51 88.9 0)
+			(at 142.24 97.79 0)
 			(hide yes)
 			(show_name no)
@@
 		)
 		(property "Value" "GND"
-			(at 143.51 90.17 0)
+			(at 143.764 93.218 0)
 			(show_name no)
 			(do_not_autoplace no)
@@
 					(size 1.27 1.27)
 				)
+				(justify left)
 			)
 		)
 		(property "Footprint" ""
-			(at 143.51 95.25 0)
+			(at 142.24 91.44 0)
 			(hide yes)
 			(show_name no)
@@
 		)
 		(property "Datasheet" ""
-			(at 143.51 95.25 0)
+			(at 142.24 91.44 0)
 			(hide yes)
 			(show_name no)
@@
 		)
 		(property "Description" "Power symbol creates a global label with name \"GND\" , ground"
-			(at 143.51 95.25 0)
+			(at 142.24 91.44 0)
 			(hide yes)
 			(show_name no)
@@
 		)
 		(instances
+			(project "Clock PCB"
+				(path "/7f3c47f2-1a05-49da-84f6-af3328144f29"
+					(reference "#PWR065")
+					(unit 1)
+				)
+			)
 			(project "StockfishChess"
 				(path "/e9cb1197-186c-4036-91fc-6928f1600b5f/83544a14-6c08-41fb-841d-407afd354856"
@@
 		)
 		(instances
+			(project "Clock PCB"
+				(path "/7f3c47f2-1a05-49da-84f6-af3328144f29"
+					(reference "J7")
+					(unit 1)
+				)
+			)
 			(project "StockfishChess"
 				(path "/e9cb1197-186c-4036-91fc-6928f1600b5f/83544a14-6c08-41fb-841d-407afd354856"
@@
 		)
 		(instances
+			(project "Clock PCB"
+				(path "/7f3c47f2-1a05-49da-84f6-af3328144f29"
+					(reference "R16")
+					(unit 1)
+				)
+			)
 			(project "StockfishChess"
 				(path "/e9cb1197-186c-4036-91fc-6928f1600b5f/83544a14-6c08-41fb-841d-407afd354856"
@@
 		)
 		(instances
+			(project "Clock PCB"
+				(path "/7f3c47f2-1a05-49da-84f6-af3328144f29"
+					(reference "R19")
+					(unit 1)
+				)
+			)
 			(project "StockfishChess"
 				(path "/e9cb1197-186c-4036-91fc-6928f1600b5f/83544a14-6c08-41fb-841d-407afd354856"
@@
 		)
 		(instances
+			(project "Clock PCB"
+				(path "/7f3c47f2-1a05-49da-84f6-af3328144f29"
+					(reference "S3")
+					(unit 1)
+				)
+			)
 			(project "StockfishChess"
 				(path "/e9cb1197-186c-4036-91fc-6928f1600b5f/83544a14-6c08-41fb-841d-407afd354856"
@@
 			)
 		)
-		(property "Value" "OLED_128X64_1.3_I2C"
+		(property "Value" "OLED_128X32_2.23_I2C"
 			(at 163.83 124.46 0)
 			(show_name no)
@@
 			)
 		)
-		(property "Footprint" "OLED_128X64_1.3_I2C:LCD_OLED_128X64_1.3_I2C"
+		(property "Footprint" "OLED_128X64_1.3_I2C:LCD_OLED_128X32_2.23_I2C"
 			(at 163.83 111.76 0)
 			(hide yes)
@@
 		)
 		(instances
+			(project "Clock PCB"
+				(path "/7f3c47f2-1a05-49da-84f6-af3328144f29"
+					(reference "DS2")
+					(unit 1)
+				)
+			)
 			(project "StockfishChess"
 				(path "/e9cb1197-186c-4036-91fc-6928f1600b5f/83544a14-6c08-41fb-841d-407afd354856"
@@
 		)
 		(instances
+			(project "Clock PCB"
+				(path "/7f3c47f2-1a05-49da-84f6-af3328144f29"
+					(reference "R17")
+					(unit 1)
+				)
+			)
 			(project "StockfishChess"
 				(path "/e9cb1197-186c-4036-91fc-6928f1600b5f/83544a14-6c08-41fb-841d-407afd354856"
@@
 		)
 		(instances
+			(project "Clock PCB"
+				(path "/7f3c47f2-1a05-49da-84f6-af3328144f29"
+					(reference "10uF7")
+					(unit 1)
+				)
+			)
 			(project "StockfishChess"
 				(path "/e9cb1197-186c-4036-91fc-6928f1600b5f/83544a14-6c08-41fb-841d-407afd354856"
@@
 		)
 		(instances
+			(project "Clock PCB"
+				(path "/7f3c47f2-1a05-49da-84f6-af3328144f29"
+					(reference "R18")
+					(unit 1)
+				)
+			)
 			(project "StockfishChess"
 				(path "/e9cb1197-186c-4036-91fc-6928f1600b5f/83544a14-6c08-41fb-841d-407afd354856"
@@
 		)
 		(instances
+			(project "Clock PCB"
+				(path "/7f3c47f2-1a05-49da-84f6-af3328144f29"
+					(reference "#PWR074")
+					(unit 1)
+				)
+			)
 			(project "StockfishChess"
 				(path "/e9cb1197-186c-4036-91fc-6928f1600b5f/83544a14-6c08-41fb-841d-407afd354856"
@@
 		)
 		(instances
+			(project "Clock PCB"
+				(path "/7f3c47f2-1a05-49da-84f6-af3328144f29"
+					(reference "S4")
+					(unit 1)
+				)
+			)
 			(project "StockfishChess"
 				(path "/e9cb1197-186c-4036-91fc-6928f1600b5f/83544a14-6c08-41fb-841d-407afd354856"
@@
 		)
 		(instances
+			(project "Clock PCB"
+				(path "/7f3c47f2-1a05-49da-84f6-af3328144f29"
+					(reference "#PWR066")
+					(unit 1)
+				)
+			)
 			(project "StockfishChess"
 				(path "/e9cb1197-186c-4036-91fc-6928f1600b5f/83544a14-6c08-41fb-841d-407afd354856"
@@
 		)
 	)
+	(sheet_instances
+		(path "/"
+			(page "1")
+		)
+	)
+	(embedded_fonts no)
 )
