File: Hardware/KiCad/Schematic-PCB/Master Chess Board/Upper PCB.kicad_pcb (KiCad board)
At the start: 4 copper layers, 288 x 288 mm, 153 parts, among them J3 ZF1-15-02-X-WT-X, U10 74HC165BQ_115, U100 AH1806-W-7, U101 AH1806-W-7, U102 AH1806-W-7, U103 AH1806-W-7, U104 AH1806-W-7, U105 AH1806-W-7, U106 AH1806-W-7, U107 AH1806-W-7, U108 AH1806-W-7, U109 AH1806-W-7, U11 74HC165BQ_115, U110 AH1806-W-7, U111 AH1806-W-7, U112 AH1806-W-7, U113 AH1806-W-7, U114 AH1806-W-7, U115 AH1806-W-7, U116 AH1806-W-7, U117 AH1806-W-7, U118 AH1806-W-7, U119 AH1806-W-7, U12 74HC165BQ_115, U120 AH1806-W-7, U121 AH1806-W-7, U122 AH1806-W-7, U123 AH1806-W-7, U124 AH1806-W-7, U125 AH1806-W-7, U126 AH1806-W-7, U127 AH1806-W-7, U128 AH1806-W-7, U129 AH1806-W-7, U13 74HC165BQ_115, U130 AH1806-W-7, U131 AH1806-W-7, U132 AH1806-W-7, U133 AH1806-W-7, U134 AH1806-W-7, U135 AH1806-W-7, U136 AH1806-W-7, U137 AH1806-W-7, U138 AH1806-W-7, U139 AH1806-W-7, U14 APA102C, U140 AH1806-W-7, U141 AH1806-W-7, U142 AH1806-W-7, U15 APA102C, U16 APA102C, U17 APA102C, U18 APA102C, U19 APA102C, U20 APA102C, U21 APA102C, U22 APA102C, U23 APA102C, U24 APA102C, U25 APA102C, U26 APA102C, U27 APA102C, U28 APA102C, U29 APA102C, U30 APA102C, U31 APA102C, U32 APA102C, U33 APA102C, U34 APA102C, U35 APA102C, U36 APA102C, U37 APA102C, U38 APA102C, U39 APA102C, U40 APA102C, U41 APA102C, U42 APA102C, U43 APA102C, U44 APA102C, U45 APA102C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

Commit message: Added pulups to hall effect
Parts:
- added 10Kohm: R_0402_1005Metric, Resistor_SMD:R_0402_1005Metric, F.Cu at (369.8, 119.7)
- added 10Kohm: R_0402_1005Metric, Resistor_SMD:R_0402_1005Metric, F.Cu at (156.2, 328.3)
- added 10Kohm: R_0402_1005Metric, Resistor_SMD:R_0402_1005Metric, F.Cu at (333.1, 156.1)
- added 10Kohm: R_0402_1005Metric, Resistor_SMD:R_0402_1005Metric, F.Cu at (405.9, 119.3)
- added 10Kohm: R_0402_1005Metric, Resistor_SMD:R_0402_1005Metric, F.Cu at (366.9, 294.2)
- added 10Kohm: R_0402_1005Metric, Resistor_SMD:R_0402_1005Metric, F.Cu at (153.7, 256.5)
- added 10Kohm: R_0402_1005Metric, Resistor_SMD:R_0402_1005Metric, F.Cu at (369.7, 191.5)
- added 10Kohm: R_0402_1005Metric, Resistor_SMD:R_0402_1005Metric, F.Cu at (155.7, 119.9)
- added 10Kohm: R_0402_1005Metric, Resistor_SMD:R_0402_1005Metric, F.Cu at (403.9, 330.2)
- added 10Kohm: R_0402_1005Metric, Resistor_SMD:R_0402_1005Metric, F.Cu at (262.8, 83.9)
- added 10Kohm: R_0402_1005Metric, Resistor_SMD:R_0402_1005Metric, F.Cu at (297.8, 191.9)
- added 10Kohm: R_0402_1005Metric, Resistor_SMD:R_0402_1005Metric, F.Cu at (227.2, 120.2)
- added 10Kohm: R_0402_1005Metric, Resistor_SMD:R_0402_1005Metric, F.Cu at (331.3, 222.4)
- added 10Kohm: R_0402_1005Metric, Resistor_SMD:R_0402_1005Metric, F.Cu at (223.4, 222.5)
- added 10Kohm: R_0402_1005Metric, Resistor_SMD:R_0402_1005Metric, F.Cu at (403.4, 258.2)
- added 10Kohm: R_0402_1005Metric, Resistor_SMD:R_0402_1005Metric, F.Cu at (405.8, 155.3)
- added 10Kohm: R_0402_1005Metric, Resistor_SMD:R_0402_1005Metric, F.Cu at (405.4, 83.2)
- added 10Kohm: R_0402_1005Metric, Resistor_SMD:R_0402_1005Metric, F.Cu at (155.9, 220.2)
- added 10Kohm: R_0402_1005Metric, Resistor_SMD:R_0402_1005Metric, F.Cu at (190.5, 192.4)
- added 10Kohm: R_0402_1005Metric, Resistor_SMD:R_0402_1005Metric, F.Cu at (259.4, 330.1)
- added 10Kohm: R_0402_1005Metric, Resistor_SMD:R_0402_1005Metric, F.Cu at (259.4, 294.2)
- added 10Kohm: R_0402_1005Metric, Resistor_SMD:R_0402_1005Metric, F.Cu at (333.8, 84.6)
- added 10Kohm: R_0402_1005Metric, Resistor_SMD:R_0402_1005Metric, F.Cu at (155.7, 155.3)
- added 10Kohm: R_0402_1005Metric, Resistor_SMD:R_0402_1005Metric, F.Cu at (262.8, 120.1)
- added 10Kohm: R_0402_1005Metric, Resistor_SMD:R_0402_1005Metric, F.Cu at (227.2, 191.5)
- added 10Kohm: R_0402_1005Metric, Resistor_SMD:R_0402_1005Metric, F.Cu at (295.2, 330.1)
- added 10Kohm: R_0402_1005Metric, Resistor_SMD:R_0402_1005Metric, F.Cu at (188.4, 222.2)
- added 10Kohm: R_0402_1005Metric, Resistor_SMD:R_0402_1005Metric, F.Cu at (367.2, 330.2)
- added 10Kohm: R_0402_1005Metric, Resistor_SMD:R_0402_1005Metric, F.Cu at (187.7, 294.1)
- added 10Kohm: R_0402_1005Metric, Resistor_SMD:R_0402_1005Metric, F.Cu at (190.5, 83.5)
- added 10Kohm: R_0402_1005Metric, Resistor_SMD:R_0402_1005Metric, F.Cu at (187.9, 258.2)
- added 10Kohm: R_0402_1005Metric, Resistor_SMD:R_0402_1005Metric, F.Cu at (191.1, 120.2)
- added 10Kohm: R_0402_1005Metric, Resistor_SMD:R_0402_1005Metric, F.Cu at (294.6, 294.2)
- added 10Kohm: R_0402_1005Metric, Resistor_SMD:R_0402_1005Metric, F.Cu at (297.4, 120.5)
- added 10Kohm: R_0402_1005Metric, Resistor_SMD:R_0402_1005Metric, F.Cu at (223.5, 294.2)
- added 10Kohm: R_0402_1005Metric, Resistor_SMD:R_0402_1005Metric, F.Cu at (330.8, 258.3)
- added 10Kohm: R_0402_1005Metric, Resistor_SMD:R_0402_1005Metric, F.Cu at (227.6, 155.7)
- added 10Kohm: R_0402_1005Metric, Resistor_SMD:R_0402_1005Metric, F.Cu at (263.0, 191.5)
- added 10Kohm: R_0402_1005Metric, Resistor_SMD:R_0402_1005Metric, F.Cu at (369.0, 155.6)
- added 10Kohm: R_0402_1005Metric, Resistor_SMD:R_0402_1005Metric, F.Cu at (405.5, 191.4)
- added 10Kohm: R_0402_1005Metric, Resistor_SMD:R_0402_1005Metric, F.Cu at (226.6, 84.1)
- added 10Kohm: R_0402_1005Metric, Resistor_SMD:R_0402_1005Metric, F.Cu at (153.7, 83.3)
- added 10Kohm: R_0402_1005Metric, Resistor_SMD:R_0402_1005Metric, F.Cu at (331.2, 330.1)
- added 10Kohm: R_0402_1005Metric, Resistor_SMD:R_0402_1005Metric, F.Cu at (334.3, 120.2)
- added 10Kohm: R_0402_1005Metric, Resistor_SMD:R_0402_1005Metric, F.Cu at (331.6, 294.3)
- added 10Kohm: R_0402_1005Metric, Resistor_SMD:R_0402_1005Metric, F.Cu at (155.7, 292.4)
- added 10Kohm: R_0402_1005Metric, Resistor_SMD:R_0402_1005Metric, F.Cu at (191.0, 156.6)
- added 10Kohm: R_0402_1005Metric, Resistor_SMD:R_0402_1005Metric, F.Cu at (402.6, 223.2)
- added 10Kohm: R_0402_1005Metric, Resistor_SMD:R_0402_1005Metric, F.Cu at (223.7, 330.0)
- added 10Kohm: R_0402_1005Metric, Resistor_SMD:R_0402_1005Metric, F.Cu at (403.3, 294.2)
- added 10Kohm: R_0402_1005Metric, Resistor_SMD:R_0402_1005Metric, F.Cu at (294.5, 258.2)
- added 10Kohm: R_0402_1005Metric, Resistor_SMD:R_0402_1005Metric, F.Cu at (155.6, 191.3)
- added 10Kohm: R_0402_1005Metric, Resistor_SMD:R_0402_1005Metric, F.Cu at (262.9, 156.0)
- added 10Kohm: R_0402_1005Metric, Resistor_SMD:R_0402_1005Metric, F.Cu at (333.3, 192.1)
- added 10Kohm: R_0402_1005Metric, Resistor_SMD:R_0402_1005Metric, F.Cu at (297.0, 155.9)
- added 10Kohm: R_0402_1005Metric, Resistor_SMD:R_0402_1005Metric, F.Cu at (369.8, 83.7)
- added 10Kohm: R_0402_1005Metric, Resistor_SMD:R_0402_1005Metric, F.Cu at (367.2, 258.4)
- added 10Kohm: R_0402_1005Metric, Resistor_SMD:R_0402_1005Metric, F.Cu at (187.6, 330.0)
- added 10Kohm: R_0402_1005Metric, Resistor_SMD:R_0402_1005Metric, F.Cu at (260.1, 222.1)
- added 10Kohm: R_0402_1005Metric, Resistor_SMD:R_0402_1005Metric, F.Cu at (259.0, 258.2)
- added 10Kohm: R_0402_1005Metric, Resistor_SMD:R_0402_1005Metric, F.Cu at (297.2, 84.7)
- added 10Kohm: R_0402_1005Metric, Resistor_SMD:R_0402_1005Metric, F.Cu at (223.6, 258.1)
- added 10Kohm: R_0402_1005Metric, Resistor_SMD:R_0402_1005Metric, F.Cu at (367.2, 222.3)
- added 10Kohm: R_0402_1005Metric, Resistor_SMD:R_0402_1005Metric, F.Cu at (294.3, 222.8)
- added 22uF: C_1206_3216Metric, Capacitor_SMD:C_1206_3216Metric, F.Cu at (300.5, 201.5)
- added 22uF: C_1206_3216Metric, Capacitor_SMD:C_1206_3216Metric, F.Cu at (295.5, 201.4)
Routing:
- net +3.3V: track 216.4 -> 458.6 mm
- net Net-(U110-OUTPUT): track 126.4 -> 133.4 mm
- net Net-(U10-D3): track 14.3 -> 20.8 mm
- net Net-(U12-D2): track 50.9 -> 57.0 mm
- net Net-(U10-D2): track 49.2 -> 55.3 mm
- net Net-(U102-OUTPUT): track 125.2 -> 131.3 mm
- net Net-(U8-D3): track 21.7 -> 27.8 mm
- net Net-(U12-D1): track 86.0 -> 91.9 mm
- net Net-(U7-D1): track 88.9 -> 94.7 mm
- net Net-(U10-D1): track 84.2 -> 90.0 mm
- net Net-(U11-D2): track 53.1 -> 58.9 mm
- net Net-(U13-D1): track 86.6 -> 92.1 mm
- net Net-(U7-D2): track 53.9 -> 59.3 mm
- net Net-(U7-D0): track 124.7 -> 130.2 mm
- net Net-(U101-OUTPUT): track 89.6 -> 95.0 mm
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